File: hardware/modem.sch (EAGLE design)
At the start: 40 parts, among them IC1 MAX3238ECDB, IC2 74LS04D, IC4 LD117ADT33TR, U1 ESP-12S

Commit message: fixed lots of minor problems of the first prototype
 - mount holes too large (3.2mm instead of 3.0mm)
 - missing keep-out around mount holes
 - resistor collides with screw in mount hole
 - button S1 collides with screw in mount hole
 - C6 and C7 were hard to solder, thermals on around caps
 - LEDs were hard to solder, thermals on VCC layer
 - debug port position and layout
 - cosmetic changes
Parts:
- removed R11, R8: (no value), rcl:R-EU_R0805
- added GND, VCC: PTR1PAD1-13, testpad:PTR1PAD1-13
- added H1, H2, H3, H4: MOUNT-HOLE3.0, holes:MOUNT-HOLE3.0
- added R33: 10k, rcl:R-EU_R0805
- C1, C2, C3, C4: value 0.1µF -> 100n
- C7: value 10µF -> 100nF
- DBG: value (none) -> PTR1PAD1-13; device pinhead:PINHD-1X2 -> testpad:PTR1PAD1-13
- R1, R2, R3, R4, R5, R6, R7: value (none) -> 820
- R10, R12, R9: value (none) -> 10k
Connections:
- removed net N$24: DBG.1, R11.2
- net !RESET: now also R33.1; no longer R3.1
- net +3V3: now also R33.2, VCC.TP; no longer R3.2
- net DEBUG: now also DBG.TP; no longer R11.1
- net GND: now also C2.2, GND.TP, S1.P; no longer C4.2, DBG.2, S1.S
- net N$10: now also R5.2; no longer R7.2
- net N$11: now also C2.1; no longer C4.1
- net N$15: now also C4.2; no longer C2.2
- net N$16: now also C4.1; no longer C2.1
- net N$17: now also R6.2; no longer R8.2
- net N$18: now also R7.2; no longer R4.2
- net N$19: now also R7.1; no longer R4.1
- net N$20: now also R6.1; no longer R8.1
- net N$21: now also R4.2; no longer R6.2
- net N$23: now also S1.S; no longer S1.P
- net N$6: now also R3.2; no longer R5.2
- net N$7: now also R3.1; no longer R5.1
- net N$8: now also R4.1; no longer R6.1
- net N$9: now also R5.1; no longer R7.1
Other:
- moved on the sheet: C2, C4, R3, R4, R5, R6, R7, S1
